File: hardware/midi-box/midi-box.kicad_sch (KiCad schematic)
At the start: 0 parts

Commit message: fix: many changes
Parts:
- added J1, J5, J6, J7: DIN-5, symbol Connector:DIN-5
- added J1, J2, J3: Screw_Terminal_01x02, symbol Connector:Screw_Terminal_01x02
- added J11: Screw_Terminal_01x03, symbol Connector:Screw_Terminal_01x03
- added J4: Raspberry_Pi_4, symbol Connector:Raspberry_Pi_4
- added R1, R10, R11, R12, R2, R3, R4, R5, R6, R7, R8, R9: 220R, symbol Device:R
Connections:
- new net: J1.4, R5.1
- new net: J1.5, R6.1
- new net: J1.1 (Pin_1), R1.1
- new net: J1.2 (Pin_2), R2.1
- new net: J2.1 (Pin_1), R3.1
- new net: J3.1 (Pin_1), R3.2, R4.2
- new net: J7.4, R12.1
- new net: J7.5, R11.1
- new net: J3.2 (Pin_2), R1.2, R2.2
- new net: J5.5, R7.1
- new net: J4.7 (GPCLK0/GPIO04), R7.2
- new net: J4.32 (GPIO12/PWM0), R6.2
- new net: J2.2 (Pin_2), R4.1
- new net: J4.1 (3V3), J4.17 (3V3)
- new net: J4.24 (~{CE0}_SPI0/GPIO08), R9.2
- new net: J4.8 (GPIO14/UART_TXD), R11.2
- new net: J6.4, R10.1
- new net: J6.5, R9.1
- new net: J5.4, R8.1
- new net +5V: J4.2 (5V), J4.4 (5V), R10.2, R12.2, R5.2, R8.2
- new net GND: J4.14 (GND), J4.20 (GND), J4.25 (GND), J4.30 (GND), J4.34 (GND), J4.39 (GND), J4.6 (GND), J4.9 (GND)
Other:
- title: (none) -> Midi Box
